Commit message: update 26/07

File: Robot/Simulation/solo12.urdf (robot description, URDF)
Before this commit: robot Solo12, 13 links, 12 joints
Links:
- removed link Hip_FL
- removed link Hip_FR
- removed link Hip_HL
- removed link Hip_HR
- added link Abduction_FL, mass 0.2; collision mesh filename=solo12_hip_fe_fl.stl; visual mesh filename=solo12_hip_fe_fl.stl
- added link Abduction_FR, mass 0.14196048; collision mesh filename=solo12_hip_fe_fr.stl; visual mesh filename=solo12_hip_fe_fr.stl
- added link Abduction_HL, mass 0.2; collision mesh filename=solo12_hip_fe_hl.stl; visual mesh filename=solo12_hip_fe_hl.stl
- added link Abduction_HR, mass 0.14196048; collision mesh filename=solo12_hip_fe_hr.stl; visual mesh filename=solo12_hip_fe_hr.stl
Joints:
- removed joint motor_lower_fl
- removed joint motor_lower_fr
- removed joint motor_lower_hl
- removed joint motor_lower_hr
- removed joint motor_upper_fl
- removed joint motor_upper_fr
- removed joint motor_upper_hl
- removed joint motor_upper_hr
- added joint motor_abduction_fl: type revolute, parent Base, child Abduction_FL, origin xyz=0.2141 0.0875 0 rpy=0 0 0, axis 1 0 0, limit lower=-1.57 upper=1.57 effort=20 velocity=100
- added joint motor_abduction_fr: type revolute, parent Base, child Abduction_FR, origin xyz=0.2141 -0.0875 0 rpy=0 0 0, axis 1 0 0, limit lower=-1.57 upper=1.57 effort=20 velocity=100
- added joint motor_abduction_hl: type revolute, parent Base, child Abduction_HL, origin xyz=-0.2141 0.0875 0 rpy=0 0 0, axis 1 0 0, limit lower=-1.57 upper=1.57 effort=20 velocity=100
- added joint motor_abduction_hr: type revolute, parent Base, child Abduction_HR, origin xyz=-0.2141 -0.0875 0 rpy=0 0 0, axis 1 0 0, limit lower=-1.57 upper=1.57 effort=20 velocity=100
- added joint motor_knee_fl: type revolute, parent Upper_FL, child Lower_FL, origin xyz=0 0.03745 -0.16 rpy=0 0 0, axis 0 -1 0, limit lower=-1.57 upper=1.57 effort=20 velocity=100
- added joint motor_knee_fr: type revolute, parent Upper_FR, child Lower_FR, origin xyz=0 -0.03745 -0.16 rpy=0 0 0, axis 0 -1 0, limit lower=-1.57 upper=1.57 effort=20 velocity=100
- added joint motor_knee_hl: type revolute, parent Upper_HL, child Lower_HL, origin xyz=0 0.03745 -0.16 rpy=0 0 0, axis 0 -1 0, limit lower=-1.57 upper=1.57 effort=20 velocity=100
- added joint motor_knee_hr: type revolute, parent Upper_HR, child Lower_HR, origin xyz=0 -0.03745 -0.16 rpy=0 0 0, axis 0 -1 0, limit lower=-1.57 upper=1.57 effort=20 velocity=100
- joint motor_hip_fl: axis 1 0 0 -> 0 -1 0; child Hip_FL -> Upper_FL; origin xyz=0.2141 0.0875 0 rpy=0 0 0 -> xyz=-0.0195 0.014 0 rpy=0 0 0; parent Base -> Abduction_FL
- joint motor_hip_fr: axis 1 0 0 -> 0 -1 0; child Hip_FR -> Upper_FR; origin xyz=0.2141 -0.0875 0 rpy=0 0 0 -> xyz=-0.0195 -0.014 0 rpy=0 0 0; parent Base -> Abduction_FR
- joint motor_hip_hl: axis 1 0 0 -> 0 -1 0; child Hip_HL -> Upper_HL; origin xyz=-0.2141 0.0875 0 rpy=0 0 0 -> xyz=0.0195 0.014 0 rpy=0 0 0; parent Base -> Abduction_HL
- joint motor_hip_hr: axis 1 0 0 -> 0 -1 0; child Hip_HR -> Upper_HR; origin xyz=-0.2141 -0.0875 0 rpy=0 0 0 -> xyz=0.0195 -0.014 0 rpy=0 0 0; parent Base -> Abduction_HR

Commit message: add some bugs

File: Robot/Simulation/solo12.urdf (robot description, URDF)
Before this commit: robot Solo12, 13 links, 12 joints
Joints:
- joint motor_abduction_fl: limit lower=-1.57 upper=1.57 effort=20 velocity=100 -> lower=-1.87 upper=1.87 effort=20 velocity=100
- joint motor_abduction_fr: limit lower=-1.57 upper=1.57 effort=20 velocity=100 -> lower=-1.87 upper=1.87 effort=20 velocity=100
- joint motor_abduction_hl: limit lower=-1.57 upper=1.57 effort=20 velocity=100 -> lower=-1.87 upper=1.87 effort=20 velocity=100
- joint motor_abduction_hr: limit lower=-1.57 upper=1.57 effort=20 velocity=100 -> lower=-1.87 upper=1.87 effort=20 velocity=100
- joint motor_hip_fl: limit lower=-1.57 upper=1.57 effort=20 velocity=100 -> lower=-1.87 upper=1.87 effort=20 velocity=100
- joint motor_hip_fr: limit lower=-1.57 upper=1.57 effort=20 velocity=100 -> lower=-1.87 upper=1.87 effort=20 velocity=100
- joint motor_hip_hl: limit lower=-1.57 upper=1.57 effort=20 velocity=100 -> lower=-1.87 upper=1.87 effort=20 velocity=100
- joint motor_hip_hr: limit lower=-1.57 upper=1.57 effort=20 velocity=100 -> lower=-1.87 upper=1.87 effort=20 velocity=100
- joint motor_knee_fl: limit lower=-1.57 upper=1.57 effort=20 velocity=100 -> lower=-1.87 upper=1.87 effort=20 velocity=100
- joint motor_knee_fr: limit lower=-1.57 upper=1.57 effort=20 velocity=100 -> lower=-1.87 upper=1.87 effort=20 velocity=100
- joint motor_knee_hl: limit lower=-1.57 upper=1.57 effort=20 velocity=100 -> lower=-1.87 upper=1.87 effort=20 velocity=100
- joint motor_knee_hr: limit lower=-1.57 upper=1.57 effort=20 velocity=100 -> lower=-1.87 upper=1.87 effort=20 velocity=100

Commit message: fix limit motion, position control

File: Robot/Simulation/solo12.urdf (robot description, URDF)
Before this commit: robot Solo12, 13 links, 12 joints
Joints:
- joint motor_hip_fl: limit lower=-1.87 upper=1.87 effort=20 velocity=100 -> lower=-3.14 upper=3.14 effort=20 velocity=100
- joint motor_hip_fr: limit lower=-1.87 upper=1.87 effort=20 velocity=100 -> lower=-3.14 upper=3.14 effort=20 velocity=100
- joint motor_hip_hl: limit lower=-1.87 upper=1.87 effort=20 velocity=100 -> lower=-3.14 upper=3.14 effort=20 velocity=100
- joint motor_hip_hr: limit lower=-1.87 upper=1.87 effort=20 velocity=100 -> lower=-3.14 upper=3.14 effort=20 velocity=100
- joint motor_knee_fl: limit lower=-1.87 upper=1.87 effort=20 velocity=100 -> lower=-3.14 upper=3.14 effort=20 velocity=100
- joint motor_knee_fr: limit lower=-1.87 upper=1.87 effort=20 velocity=100 -> lower=-3.14 upper=3.14 effort=20 velocity=100
- joint motor_knee_hl: limit lower=-1.87 upper=1.87 effort=20 velocity=100 -> lower=-3.14 upper=3.14 effort=20 velocity=100
- joint motor_knee_hr: limit lower=-1.87 upper=1.87 effort=20 velocity=100 -> lower=-3.14 upper=3.14 effort=20 velocity=100

Commit message: update urdf

File: Robot/Simulation/solo12.urdf (robot description, URDF)
Before this commit: robot Solo12, 13 links, 12 joints
Links:
- link Abduction_FL: mass 0.2 -> 0.14196048
- link Abduction_HL: mass 0.2 -> 0.14196048
