Commit message: update new urdf

File: a1_custom/a1.urdf (robot description, URDF)
Before this commit: robot a1_description, 26 links, 25 joints
Links:
- removed link red_sphere_1
- removed link red_sphere_2
- removed link red_sphere_3
- removed link red_sphere_4
Joints:
- removed joint red_sphere_1_to_base
- removed joint red_sphere_2_to_base
- removed joint red_sphere_3_to_base
- removed joint red_sphere_4_to_base

Commit message: update kinematic

File: a1_custom/a1.urdf (robot description, URDF)
Before this commit: robot a1_description, 22 links, 21 joints
Links:
- added link sphere_1, mass 0.001; collision sphere radius=0.014; visual sphere radius=0.014
- added link sphere_2, mass 0.001; collision sphere radius=0.014; visual sphere radius=0.014
- added link sphere_3, mass 0.001; collision sphere radius=0.014; visual sphere radius=0.014
- added link sphere_4, mass 0.001; collision sphere radius=0.014; visual sphere radius=0.014
Joints:
- added joint joint_sphere_1_base: type fixed, parent trunk, child sphere_1, origin xyz=0.14544602 -0.2035496 -0.21173298 rpy=0 0 0
- added joint joint_sphere_2_base: type fixed, parent trunk, child sphere_2, origin xyz=0.14544602 0.1991776 -0.21173298 rpy=0 0 0
- added joint joint_sphere_3_base: type fixed, parent trunk, child sphere_3, origin xyz=-0.22055398 -0.2035496 -0.21173298 rpy=0 0 0
- added joint joint_sphere_4_base: type fixed, parent trunk, child sphere_4, origin xyz=-0.22055398 0.1991776 -0.21173298 rpy=0 0 0

File: motion_imitation/robots/simulation/solo12.urdf (robot description, URDF)
Before this commit: robot solo12, 13 links, 12 joints
Links:
- added link sphere_1; visual sphere radius=0.012
- added link sphere_2; visual sphere radius=0.012
Joints:
- added joint joint_sphere_1_base: type fixed, parent base, child sphere_1, origin xyz=0.19377034 -0.27476112 -0.16903458 rpy=0 0 0
- added joint joint_sphere_2_base: type fixed, parent base, child sphere_2, origin xyz=0.19377034 0.27476112 -0.16903458 rpy=0 0 0
