Commit message: update new urdf

File: motion_imitation/robots/simulation/solo12.urdf (robot description, URDF)
Before this commit: robot Solo12, 13 links, 12 joints
Links:
- removed link Abduction_FL
- removed link Abduction_FR
- removed link Abduction_HL
- removed link Abduction_HR
- removed link Base
- removed link Lower_FL
- removed link Lower_FR
- removed link Lower_HL
- removed link Lower_HR
- removed link Upper_FL
- removed link Upper_FR
- removed link Upper_HL
- removed link Upper_HR
- added link abduction_FL, mass 0.696; collision mesh filename=abduction.stl; visual mesh filename=abduction.stl scale=1 1 1
- added link abduction_FR, mass 0.696; collision mesh filename=abduction.stl; visual mesh filename=abduction.stl scale=1 1 1
- added link abduction_HL, mass 0.696; collision mesh filename=abduction.stl; visual mesh filename=abduction.stl scale=1 1 1
- added link abduction_HR, mass 0.696; collision mesh filename=abduction.stl; visual mesh filename=abduction.stl scale=1 1 1
- added link base, mass 4.713; collision box size=0.4 0.105 0.06; visual mesh filename=base.STL scale=1 1 1
- added link lower_FL, mass 0.166; collision mesh filename=lower.STL; visual mesh filename=lower.STL scale=1 1 1
- added link lower_FR, mass 0.166; collision mesh filename=lower.STL; visual mesh filename=lower.STL scale=1 1 1
- added link lower_HL, mass 0.166; collision mesh filename=lower.STL; visual mesh filename=lower.STL scale=1 1 1
- added link lower_HR, mass 0.166; collision mesh filename=lower.STL; visual mesh filename=lower.STL scale=1 1 1
- added link upper_FL, mass 1.013; collision mesh filename=upper.stl; visual mesh filename=upper.stl scale=1 1 1
- added link upper_FR, mass 1.013; collision mesh filename=upper.stl; visual mesh filename=upper.stl scale=1 1 1
- added link upper_HL, mass 1.013; collision mesh filename=upper.stl; visual mesh filename=upper.stl scale=1 1 1
- added link upper_HR, mass 1.013; collision mesh filename=upper.stl; visual mesh filename=upper.stl scale=1 1 1
Joints:
- joint motor_abduction_fl: child Abduction_FL -> abduction_FL; limit lower=-1.87 upper=1.87 effort=20 velocity=100 -> lower=-0.802851455917 upper=0.802851455917 effort=20 velocity=52.4; parent Base -> base
- joint motor_abduction_fr: child Abduction_FR -> abduction_FR; limit lower=-1.87 upper=1.87 effort=20 velocity=100 -> lower=-0.802851455917 upper=0.802851455917 effort=20 velocity=52.4; parent Base -> base
- joint motor_abduction_hl: child Abduction_HL -> abduction_HL; limit lower=-1.87 upper=1.87 effort=20 velocity=100 -> lower=-0.802851455917 upper=0.802851455917 effort=20 velocity=52.4; parent Base -> base
- joint motor_abduction_hr: child Abduction_HR -> abduction_HR; limit lower=-1.87 upper=1.87 effort=20 velocity=100 -> lower=-0.802851455917 upper=0.802851455917 effort=20 velocity=52.4; parent Base -> base
- joint motor_hip_fl: axis 0 -1 0 -> 0 1 0; child Upper_FL -> upper_FL; limit lower=-3.14 upper=3.14 effort=20 velocity=100 -> lower=-1.0471975512 upper=4.18879020479 effort=55 velocity=28.6; parent Abduction_FL -> abduction_FL
- joint motor_hip_fr: axis 0 -1 0 -> 0 1 0; child Upper_FR -> upper_FR; limit lower=-3.14 upper=3.14 effort=20 velocity=100 -> lower=-1.0471975512 upper=4.18879020479 effort=55 velocity=28.6; parent Abduction_FR -> abduction_FR
- joint motor_hip_hl: axis 0 -1 0 -> 0 1 0; child Upper_HL -> upper_HL; limit lower=-3.14 upper=3.14 effort=20 velocity=100 -> lower=-1.0471975512 upper=4.18879020479 effort=55 velocity=28.6; parent Abduction_HL -> abduction_HL
- joint motor_hip_hr: axis 0 -1 0 -> 0 1 0; child Upper_HR -> upper_HR; limit lower=-3.14 upper=3.14 effort=20 velocity=100 -> lower=-1.0471975512 upper=4.18879020479 effort=55 velocity=28.6; parent Abduction_HR -> abduction_HR
- joint motor_knee_fl: axis 0 -1 0 -> 0 1 0; child Lower_FL -> lower_FL; limit lower=-3.14 upper=3.14 effort=20 velocity=100 -> lower=-2.69653369433 upper=-0.916297857297 effort=55 velocity=28.6; parent Upper_FL -> upper_FL
- joint motor_knee_fr: axis 0 -1 0 -> 0 1 0; child Lower_FR -> lower_FR; limit lower=-3.14 upper=3.14 effort=20 velocity=100 -> lower=-2.69653369433 upper=-0.916297857297 effort=55 velocity=28.6; parent Upper_FR -> upper_FR
- joint motor_knee_hl: axis 0 -1 0 -> 0 1 0; child Lower_HL -> lower_HL; limit lower=-3.14 upper=3.14 effort=20 velocity=100 -> lower=-2.69653369433 upper=-0.916297857297 effort=55 velocity=28.6; parent Upper_HL -> upper_HL
- joint motor_knee_hr: axis 0 -1 0 -> 0 1 0; child Lower_HR -> lower_HR; limit lower=-3.14 upper=3.14 effort=20 velocity=100 -> lower=-2.69653369433 upper=-0.916297857297 effort=55 velocity=28.6; parent Upper_HR -> upper_HR

Commit message: update

File: motion_imitation/robots/simulation/solo12.urdf (robot description, URDF)
Before this commit: robot solo12, 15 links, 14 joints
Links:
- removed link sphere_1
- removed link sphere_2
Joints:
- removed joint joint_sphere_1_base
- removed joint joint_sphere_2_base
- joint motor_abduction_fl: limit lower=-0.802851455917 upper=0.802851455917 effort=20 velocity=52.4 -> lower=-1.87 upper=1.87 effort=20 velocity=52.4
- joint motor_abduction_fr: limit lower=-0.802851455917 upper=0.802851455917 effort=20 velocity=52.4 -> lower=-1.87 upper=1.87 effort=20 velocity=52.4
- joint motor_abduction_hl: limit lower=-0.802851455917 upper=0.802851455917 effort=20 velocity=52.4 -> lower=-1.87 upper=1.87 effort=20 velocity=52.4
- joint motor_abduction_hr: limit lower=-0.802851455917 upper=0.802851455917 effort=20 velocity=52.4 -> lower=-1.87 upper=1.87 effort=20 velocity=52.4
- joint motor_hip_fl: limit lower=-1.0471975512 upper=4.18879020479 effort=55 velocity=28.6 -> lower=-3.14 upper=3.14 effort=55 velocity=28.6
- joint motor_hip_fr: limit lower=-1.0471975512 upper=4.18879020479 effort=55 velocity=28.6 -> lower=-3.14 upper=3.14 effort=55 velocity=28.6
- joint motor_hip_hl: limit lower=-1.0471975512 upper=4.18879020479 effort=55 velocity=28.6 -> lower=-3.14 upper=3.14 effort=55 velocity=28.6
- joint motor_hip_hr: limit lower=-1.0471975512 upper=4.18879020479 effort=55 velocity=28.6 -> lower=-3.14 upper=3.14 effort=55 velocity=28.6
- joint motor_knee_fl: limit lower=-2.69653369433 upper=-0.916297857297 effort=55 velocity=28.6 -> lower=-3.14 upper=3.14 effort=55 velocity=28.6
- joint motor_knee_fr: limit lower=-2.69653369433 upper=-0.916297857297 effort=55 velocity=28.6 -> lower=-3.14 upper=3.14 effort=55 velocity=28.6
- joint motor_knee_hl: limit lower=-2.69653369433 upper=-0.916297857297 effort=55 velocity=28.6 -> lower=-3.14 upper=3.14 effort=55 velocity=28.6
- joint motor_knee_hr: limit lower=-2.69653369433 upper=-0.916297857297 effort=55 velocity=28.6 -> lower=-3.14 upper=3.14 effort=55 velocity=28.6
